File: LEDController.brd (EAGLE design)
At the start: 25 x 50 mm, 30 parts, among them IC1 LP298XS, J1 POWER_JACKPTH, U1 CC3000, U2 ATTINY84

Commit message: Update
Update before submission to fab
Parts:
- removed C16: 10uF, SparkFun-Capacitors:0603-CAP
- removed IC1: LP298XS, adafruit:SOT23-5L
- removed U$1: AVR_MINI_PROGSMD, SparkFun-Connectors:AVR_MINI_PROG
- removed U$2: ANTENNA22500AT44M0400, SparkFun-RF:ANTENNA-CHIP_2500AT44M0400
- added C1: 1.0uF, SparkFun-Capacitors:0603-CAP
- added JP2: AVR_MINI_PROGSMD, SparkFun-Connectors:AVR_MINI_PROG
- added U3: CC3000, SparkFun-RF:QFN-46_CC3000
- added X1: (no value), SparkFun-FreqCtrl:CRYSTAL-SMD-5X3
- C10: value 1.0uF -> 10uF
- C11: value 20 pF -> 2.2 pF
- C12: value 20 pF -> 10 pF
- C13: value 1.0uF -> 0.1uF
- C14: value 10uF -> 0.1uF
- C2: value 0.1uF -> 10uF
- C3: value 0.1uF -> 1.0uF
- C4: value 1.0uF -> 10nF
- C7: value 10nF -> 20 pF
- C8: value 10 pF -> 20 pF
- C9: value 2.2 pF -> 1.0uF
- U1: value CC3000 -> ATTINY84; device SparkFun-RF:QFN-46_CC3000 -> SparkFun-DigitalIC:SO14
- U2: value ATTINY84 -> LP298XS; device SparkFun-DigitalIC:SO14 -> adafruit:SOT23-5L
- Y1: value (none) -> ANTENNA22500AT44M0400; device SparkFun-FreqCtrl:CRYSTAL-SMD-5X3 -> SparkFun-RF:ANTENNA-CHIP_2500AT44M0400
- moved C9 30.8 mm to (17.1, 33.7), turned to 90 degrees
- moved Y1 30.6 mm to (5.71, 3.17), turned to 180 degrees
- moved C12 30.5 mm to (18.2, 7.49), turned to 90 degrees
- moved C8 30.5 mm to (6.35, 35.6), turned to 270 degrees
- moved C11 29.2 mm to (12.5, 3.17), turned to 0 degrees
- moved C4 25.9 mm to (16.5, 40.6), turned to 0 degrees
- moved C14 21.1 mm to (6.99, 19.7)
- moved C3 20.2 mm to (21.6, 33.7)
- moved C2 19.7 mm to (23.5, 33.7), turned to 90 degrees
- moved C15 19.6 mm to (6.99, 16.5), turned to 270 degrees
- moved C7 18.8 mm to (6.35, 31.8), turned to 90 degrees
- moved C13 17.7 mm to (6.99, 22.9), turned to 270 degrees
- moved U1 14.7 mm to (10.8, 32.4), turned to 270 degrees
- moved U2 9.71 mm to (20.3, 30.5), turned to 90 degrees
- moved C10 8.28 mm to (19.1, 33.7), turned to 90 degrees
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- renumbered R4 to R2, R5 to R1
Connections:
- net !RESET: now also JP2.3, U1.4; no longer U$1.3, U2.4
- net 3.3V: now also C1.1, C13.1, C14.1, C9.1, JP2.1, U1.1, U2.5, U3.P$19, U3.P$23; no longer C16.1, C2.1, C3.1, C4.1, IC1.5, U$1.1, U1.P$19, U1.P$23, U2.1
- net CS_WIFI: now also U1.6, U3.P$12; no longer U1.P$12, U2.6
- net EN_WIFI: now also U1.5, U3.P$26; no longer U1.P$26, U2.5
- net GND: now also C1.2, C7.1, C8.1, C9.2, JP2.2, U1.14, U2.2, U3.GND@37, U3.GND@38, U3.GND@39, U3.GND@40, U3.GND@41, U3.GND@42, U3.GND@43, U3.GND@44, U3.GND@45, U3.GND@46, U3.P$1, U3.P$10, U3.P$11, U3.P$16, U3.P$18, U3.P$20, U3.P$21, U3.P$22, U3.P$25, U3.P$31, U3.P$32, U3.P$33, U3.P$34, U3.P$36, U3.P$9; no longer C11.1, C12.1, C16.2, C7.2, IC1.2, U$1.2, U1.GND@37, U1.GND@38, U1.GND@39, U1.GND@40, U1.GND@41, U1.GND@42, U1.GND@43, U1.GND@44, U1.GND@45, U1.GND@46, U1.P$1, U1.P$10, U1.P$11, U1.P$16, U1.P$18, U1.P$20, U1.P$21, U1.P$22, U1.P$25, U1.P$31, U1.P$32, U1.P$33, U1.P$34, U1.P$36, U1.P$9, U2.14
- net INT_WIFI: now also U1.10, U3.P$14; no longer U1.P$14, U2.10
- net MISO: now also JP2.6, U1.8, U3.P$13; no longer U$1.6, U1.P$13, U2.8
- net MOSI: now also JP2.4, U1.7, U3.P$15; no longer U$1.4, U1.P$15, U2.7
- net N$10: now also C11.2, C12.1; no longer C8.1, C9.2
- net N$11: now also C11.1, Y1.FEED; no longer C9.1, U$2.FEED
- net N$12: now also C7.2, U1.3, X1.1; no longer C11.2, U2.3, Y1.1
- net N$13: now also C8.2, U1.2, X1.3; no longer C12.2, U2.2, Y1.3
- net N$2: now also U3.P$27, U3.P$28; no longer U1.P$27, U1.P$28
- net N$3: now also U3.P$29, U3.P$30; no longer U1.P$29, U1.P$30
- net N$4: now also C6.1; no longer C7.1
- net N$5: now also C5.1; no longer C6.1
- net N$6: now also C4.1; no longer C5.1
- net N$8: now also U3.P$5, U3.P$7; no longer U1.P$5, U1.P$7
- net PWM_B: now also U1.11; no longer U2.11
- net PWM_G: now also U1.12; no longer U2.12
- net PWM_R: now also U1.13; no longer U2.13
- net RF_ANT: now also C12.2, U3.P$35; no longer C8.2, U1.P$35
- net SCK: now also JP2.5, U1.9, U3.P$17; no longer U$1.5, U1.P$17, U2.9
- net VIN_12V: now also C2.1, C3.1, U2.1, U2.3; no longer C13.1, C14.1, IC1.1, IC1.3
Routing:
- net MISO: track 0.00 -> 34.7 mm, vias 0 -> 1
- net SCK: track 0.00 -> 31.4 mm, vias 0 -> 1
- net EN_WIFI: track 0.00 -> 25.9 mm, vias 0 -> 2
- net MOSI: track 0.00 -> 24.7 mm, vias 0 -> 2
- net !RESET: track 0.00 -> 19.3 mm, vias 0 -> 2
- net PWM_B: track 0.00 -> 15.4 mm
- net CS_WIFI: track 0.00 -> 15.3 mm
- net GND: track 0.00 -> 14.6 mm, vias 50 -> 79
- net INT_WIFI: track 0.00 -> 11.3 mm
- net PWM_G: track 0.00 -> 11.2 mm
- net N$13: track 0.00 -> 7.67 mm
- net PWM_R: track 0.00 -> 6.93 mm
- net 3.3V: track 0.00 -> 4.57 mm, vias 2 -> 8
- net N$8: track 0.00 -> 4.45 mm
- net N$12: track 0.00 -> 4.44 mm
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- added copper zone on layer 1, net 3.3V
- added copper zone on layer 16, net 3.3V
- added copper zone on layer 1, net VIN_12V
- added copper zone on layer 16, net VIN_12V
Other:
- board text added: "JP2"
