File: LEDController.sch (EAGLE design)
At the start: 30 parts, among them IC1 LP298XS, J1 POWER_JACKPTH, U1 CC3000, U2 ATTINY84

Commit message: Update
Update before submission to fab
Parts:
- removed C16: 10uF, SparkFun-Capacitors:10UF-6.3V-20%(0603)
- removed IC1: LP298XS, adafruit:LP298XS
- removed U$2: ANTENNA22500AT44M0400, SparkFun-RF:ANTENNA22500AT44M0400
- added C1: 1.0uF, SparkFun-Capacitors:1.0UF-16V-10%(0603)
- added U3: CC3000, SparkFun-RF:CC3000
- added X1: (no value), SparkFun-FreqCtrl:CRYSTAL5X3
- C10: value 1.0uF -> 10uF; device SparkFun-Capacitors:1.0UF-16V-10%(0603) -> SparkFun-Capacitors:10UF-6.3V-20%(0603)
- C11: value 20 pF -> 2.2 pF
- C12: value 20 pF -> 10 pF
- C13: value 1.0uF -> 0.1uF; device SparkFun-Capacitors:1.0UF-16V-10%(0603) -> SparkFun-Capacitors:0.1UF-25V-5%(0603)
- C14: value 10uF -> 0.1uF; device SparkFun-Capacitors:10UF-6.3V-20%(0603) -> SparkFun-Capacitors:0.1UF-25V-5%(0603)
- C2: value 0.1uF -> 10uF; device SparkFun-Capacitors:0.1UF-25V-5%(0603) -> SparkFun-Capacitors:10UF-6.3V-20%(0603)
- C3: value 0.1uF -> 1.0uF; device SparkFun-Capacitors:0.1UF-25V-5%(0603) -> SparkFun-Capacitors:1.0UF-16V-10%(0603)
- C4: value 1.0uF -> 10nF; device SparkFun-Capacitors:1.0UF-16V-10%(0603) -> SparkFun-Capacitors:10NF/10000PF-50V-10%(0603)
- C7: value 10nF -> 20 pF; device SparkFun-Capacitors:10NF/10000PF-50V-10%(0603) -> SparkFun-Capacitors:9.0PF-50V-10%(0603)
- C8: value 10 pF -> 20 pF
- C9: value 2.2 pF -> 1.0uF; device SparkFun-Capacitors:9.0PF-50V-10%(0603) -> SparkFun-Capacitors:1.0UF-16V-10%(0603)
- U1: value CC3000 -> ATTINY84; device SparkFun-RF:CC3000 -> SparkFun-DigitalIC:ATTINY84
- U2: value ATTINY84 -> LP298XS; device SparkFun-DigitalIC:ATTINY84 -> adafruit:LP298XS
- Y1: value (none) -> ANTENNA22500AT44M0400; device SparkFun-FreqCtrl:CRYSTAL5X3 -> SparkFun-RF:ANTENNA22500AT44M0400
- renumbered R4 to R2, R5 to R1, U$1 to JP2
Connections:
- net !RESET: now also U1.(PCINT11/~RESET/DW)PB3; no longer U2.(PCINT11/~RESET/DW)PB3
- net 3.3V: now also C1.1, C13.1, C14.1, C9.1, U1.VCC, U2.VOUT, U3.VBAT_IN, U3.VIO_HOST; no longer C16.1, C2.1, C3.1, C4.1, IC1.VOUT, U1.VBAT_IN, U1.VIO_HOST, U2.VCC
- net CS_WIFI: now also U1.(PCINT7/ICP/OC0B/ADC7)PA7, U3.SPI_CS; no longer U1.SPI_CS, U2.(PCINT7/ICP/OC0B/ADC7)PA7
- net EN_WIFI: now also U1.(PCINT10/INT0/OC0A/CKOUT)PB2, U3.VBAT_SW_EN; no longer U1.VBAT_SW_EN, U2.(PCINT10/INT0/OC0A/CKOUT)PB2
- net GND: now also C1.2, C7.1, C8.1, C9.2, U1.GND, U3.EXT_32K, U3.GND@1, U3.GND@10, U3.GND@11, U3.GND@16, U3.GND@18, U3.GND@20, U3.GND@22, U3.GND@25, U3.GND@31, U3.GND@32, U3.GND@33, U3.GND@34, U3.GND@36, U3.GND@37, U3.GND@38, U3.GND@39, U3.GND@40, U3.GND@41, U3.GND@42, U3.GND@43, U3.GND@44, U3.GND@45, U3.GND@46, U3.GND@9; no longer C11.1, C12.1, C16.2, C7.2, IC1.GND, U1.EXT_32K, U1.GND@1, U1.GND@10, U1.GND@11, U1.GND@16, U1.GND@18, U1.GND@20, U1.GND@22, U1.GND@25, U1.GND@31, U1.GND@32, U1.GND@33, U1.GND@34, U1.GND@36, U1.GND@37, U1.GND@38, U1.GND@39, U1.GND@40, U1.GND@41, U1.GND@42, U1.GND@43, U1.GND@44, U1.GND@45, U1.GND@46, U1.GND@9
- net INT_WIFI: now also U1.(PCINT3/T0/ADC3)PA3, U3.SPI_IRQ; no longer U1.SPI_IRQ, U2.(PCINT3/T0/ADC3)PA3
- net MISO: now also U1.(PCINT5/OC1B/MISO/DO/ADC5)PA5, U3.SPI_DOUT; no longer U1.SPI_DOUT, U2.(PCINT5/OC1B/MISO/DO/ADC5)PA5
- net MOSI: now also U1.(PCINT6/OC1A/SDA/MOSI/ADC6)PA6, U3.SPI_DIN; no longer U1.SPI_DIN, U2.(PCINT6/OC1A/SDA/MOSI/ADC6)PA6
- net N$10: now also C11.2, C12.1; no longer C8.1, C9.2
- net N$11: now also C11.1, Y1.SIGNAL; no longer C9.1, U$2.SIGNAL
- net N$12: now also C7.2, U1.(PCINT9/XTAL2)PB1, X1.1; no longer C11.2, U2.(PCINT9/XTAL2)PB1, Y1.1
- net N$13: now also C8.2, U1.(PCINT8/XTAL1/CLKI)PB0, X1.2; no longer C12.2, U2.(PCINT8/XTAL1/CLKI)PB0, Y1.2
- net N$2: now also U3.SDA_CC3000, U3.SDA_EEPROM; no longer U1.SDA_CC3000, U1.SDA_EEPROM
- net N$3: now also U3.SCL_CC3000, U3.SCL_EEPROM; no longer U1.SCL_CC3000, U1.SCL_EEPROM
- net N$4: now also C6.1; no longer C7.1
- net N$5: now also C5.1; no longer C6.1
- net N$6: now also C4.1; no longer C5.1
- net N$8: now also U3.WL_EN1, U3.WL_EN2; no longer U1.WL_EN1, U1.WL_EN2
- net PWM_B: now also U1.(PCINT2/AIN1/ADC2)PA2; no longer U2.(PCINT2/AIN1/ADC2)PA2
- net PWM_G: now also U1.(PCINT1/AIN0/ADC1)PA1; no longer U2.(PCINT1/AIN0/ADC1)PA1
- net PWM_R: now also U1.(PCINT0/AREF/ADC0)PA0; no longer U2.(PCINT0/AREF/ADC0)PA0
- net RF_ANT: now also C12.2, U3.RF_ANT; no longer C8.2, U1.RF_ANT
- net SCK: now also U1.(PCINT4/T1/SCL/USCK/ADC4)PA4, U3.SPI_CLK; no longer U1.SPI_CLK, U2.(PCINT4/T1/SCL/USCK/ADC4)PA4
- net VIN_12V: now also C2.1, C3.1, U2.EN, U2.VIN; no longer C13.1, C14.1, IC1.EN, IC1.VIN
Other:
- moved on the sheet: C10, C11, C12, C13, C14, C15, C2, C3, C4, C5, C6, C7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
